File: PCB/usbuh.kicad_pcb (KiCad board)
At the start: 2 copper layers, 90 x 55 mm, 69 parts, among them U1 FE1.1s, U2 FE1.1s, U4 AMS1117-3.3, U5 PCM2902, Y1 12MHz, Y2 12MHz, Y3 12MHz

Commit message: Update PCB
Parts:
- added G***: LOGO, LOGO, F.Cu at (113.2, 138.2)
- C13, C15, C26, R14, R19: moved to F.Cu
- moved C13 0.58 mm to (138.6, 103.2)
- moved C15 0.56 mm to (138.6, 100.8)
- moved R14 0.56 mm to (161.6, 136.6)
- turned C26 to 0 degrees
Routing:
- net +5V: track 192.4 -> 202.8 mm, vias 13 -> 15
- net MicBias: track 40.7 -> 34.1 mm, vias 1 -> 0
- net +3V3: track 144.6 -> 146.0 mm, vias 10 -> 11
- net U1DMU: track 41.4 -> 40.8 mm
- net GND: track 381.5 -> 382.0 mm, vias 11 -> 10
- net Net-(USB_C_1-CC2): track 2.95 -> 3.38 mm, vias 1 -> 0
- net VDDI: track 45.7 -> 45.8 mm, vias 5 -> 6
- added copper zone on B.Cu, net GND
- added copper zone on F.Cu, net GND
